Commit message: Add marker trajectories. Finish detector

File: workcell_scene_description/urdf/marker.urdf.xacro (robot description, xacro)
@@ -3,5 +3,5 @@
   <!-- Marker macro model -->
   <xacro:macro name="marker" params="name parent scale *origin">
-      <joint name="${name}_joint" type="fixed">
+      <joint name="${name}_joint" type="floating">
         <xacro:insert_block name="origin" />
         <parent link="${parent}"/>
@@ -28,4 +28,5 @@
       </link>
       <gazebo reference="${name}_link">
+        <turnGravityOff>true</turnGravityOff>
       </gazebo>
     </xacro:macro>

File: workcell_scene_description/urdf/workcell.urdf.xacro (robot description, xacro)
@@ -50,6 +50,6 @@
     <!-- Marker -->
    <xacro:include filename="$(find workcell_scene_description)/urdf/marker.urdf.xacro"/>
-   <xacro:marker name="marker" parent="world" scale="1.5">
-     <origin xyz="1.25 0.25 1.5" rpy="0 0 3.14"/>
+   <xacro:marker name="marker" parent="world" scale="1">
+     <origin xyz="1.25 0.25 1.7" rpy="0 0 3.14"/>
    </xacro:marker>
 </robot>
